File: hw/2_2_4.kicad_sch (KiCad schematic)
At the start: 29 parts, among them SW4 SW_Push, U1 ATmega2560-16A, U2 AP64501SP-13

Commit message: Add LM2576S-5 to 2.3.10
Signed-off-by: ckalina <46683072+ckalina@users.noreply.github.com>
Changed lines of the file:
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@@
   (text "https://www.diodes.com/assets/Datasheets/AP64501.pdf"
     (at 180.34 109.22 0)
-    (effects (font (size 1.27 1.27)))
+    (effects (font (size 1.27 1.27)) (justify left bottom))
   )
   (label "PA0" (at 20.32 45.72 0)
