File: hw/2_2_8.kicad_sch (KiCad schematic)
At the start: 4 parts

Commit message: Add LM2576S-5 to 2.3.10
Signed-off-by: ckalina <46683072+ckalina@users.noreply.github.com>
Changed lines of the file:
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@@
   )
   (text "https://docs.broadcom.com/docs/ASMG-PT00-DS100" (at 186.69 86.36 180)
-    (effects (font (size 1.27 1.27)))
+    (effects (font (size 1.27 1.27)) (justify right bottom))
   )
   (hierarchical_label "RED" (shape input) (at 106.68 92.71 180)
